Commit message: Changes for jazzy.

File: robots/common/franka_arm.ros2_control.xacro (robot description, xacro)
@@ -18,5 +18,5 @@
           </xacro:if>
           <xacro:if value="${gazebo}">
-            <plugin>franka_ign_ros2_control/IgnitionSystem</plugin>
+            <plugin>gz_ros2_control/GazeboSimSystem</plugin>
           </xacro:if>
           <xacro:if value="${use_fake_hardware == 0 and gazebo == 0}">
@@ -53,9 +53,10 @@
       <xacro:if value="${gazebo and hand}">
         <xacro:configure_joint joint_name="${arm_id}_finger_joint1" initial_position="0.0" />
+        <joint name="${arm_id}_finger_joint2" />
       </xacro:if>
     </ros2_control>
     <xacro:if value="${gazebo}">
       <gazebo>
-        <plugin filename="franka_ign_ros2_control-system" name="ign_ros2_control::IgnitionROS2ControlPlugin">
+        <plugin filename="gz_ros2_control-system" name="gz_ros2_control::GazeboSimROS2ControlPlugin">
           <parameters>$(find franka_gazebo_bringup)/config/franka_gazebo_controllers.yaml</parameters>
         </plugin>

Commit message: Add gripper support in simulation.
Signed-off-by: Jelmer de Wolde <jelmer.de.wolde@alliander.com>

File: robots/common/franka_arm.ros2_control.xacro (robot description, xacro)
@@ -53,4 +53,8 @@
       <xacro:if value="${gazebo and hand}">
         <xacro:configure_joint joint_name="${arm_id}_finger_joint1" initial_position="0.0" />
+        <joint name="${arm_id}_finger_joint2">
+          <param name="mimic">${arm_id}_finger_joint1</param>
+          <param name="multiplier">1</param>
+        </joint>
       </xacro:if>
     </ros2_control>

Commit message: Gripper support (#1)
* Add gripper support in simulation.

Signed-off-by: Jelmer de Wolde <jelmer.de.wolde@alliander.com>

* Add option to load ign_ros2_control without gazebo.

Signed-off-by: Jelmer de Wolde <jelmer.de.wolde@alliander.com>

---------

Signed-off-by: Jelmer de Wolde <jelmer.de.wolde@alliander.com>

File: robots/common/franka_arm.ros2_control.xacro (robot description, xacro)
@@ -6,4 +6,5 @@
              use_fake_hardware:=^|false
              fake_sensor_commands:=^|false
+             ign_ros2_control:=^|false
              gazebo:=^|false
              hand:=^|false
@@ -17,8 +18,8 @@
             <param name="state_following_offset">0.0</param>
           </xacro:if>
-          <xacro:if value="${gazebo}">
-            <plugin>franka_ign_ros2_control/IgnitionSystem</plugin>
+          <xacro:if value="${gazebo or ign_ros2_control}">
+            <plugin>ign_ros2_control/IgnitionSystem</plugin>
           </xacro:if>
-          <xacro:if value="${use_fake_hardware == 0 and gazebo == 0}">
+          <xacro:if value="${use_fake_hardware == 0 and gazebo == 0 and ign_ros2_control == 0}">
             <plugin>franka_hardware/FrankaHardwareInterface</plugin>
             <param name="robot_ip">${robot_ip}</param>
@@ -31,5 +32,5 @@
             https://github.com/ros-controls/gz_ros2_control/issues/343
           -->
-          <xacro:if value="${gazebo == 0 or gazebo_effort == 1}">
+          <xacro:if value="${(gazebo == 0 and ign_ros2_control == 0) or gazebo_effort == 1}">
             <command_interface name="effort"/>
           </xacro:if>
@@ -51,11 +52,15 @@
       <xacro:configure_joint joint_name="${arm_id}_joint6" initial_position="${pi/2}"/>
       <xacro:configure_joint joint_name="${arm_id}_joint7" initial_position="${pi/4}"/>
-      <xacro:if value="${gazebo and hand}">
+      <xacro:if value="${(gazebo or ign_ros2_control) and hand}">
         <xacro:configure_joint joint_name="${arm_id}_finger_joint1" initial_position="0.0" />
+        <joint name="${arm_id}_finger_joint2">
+          <param name="mimic">${arm_id}_finger_joint1</param>
+          <param name="multiplier">1</param>
+        </joint>
       </xacro:if>
     </ros2_control>
     <xacro:if value="${gazebo}">
       <gazebo>
-        <plugin filename="franka_ign_ros2_control-system" name="ign_ros2_control::IgnitionROS2ControlPlugin">
+        <plugin filename="ign_ros2_control-system" name="ign_ros2_control::IgnitionROS2ControlPlugin">
           <parameters>$(find franka_gazebo_bringup)/config/franka_gazebo_controllers.yaml</parameters>
         </plugin>
